File: 65Percent.kicad_pcb (KiCad board)
At the start: 2 copper layers, 301 x 94.7 mm, 163 parts, among them J1 ISP Headers, J2 USB C Port, K1 KEYSW, K10 KEYSW, K11 KEYSW, K12 KEYSW, K13 KEYSW, K14 KEYSW, K15 KEYSW, K16 KEYSW, K17 KEYSW, K18 KEYSW, K19 KEYSW, K2 KEYSW, K20 KEYSW, K21 KEYSW, K22 KEYSW, K23 KEYSW, K24 KEYSW, K25 KEYSW, K26 KEYSW, K27 KEYSW, K28 KEYSW, K29 KEYSW, K3 KEYSW, K30 KEYSW, K31 KEYSW, K32 KEYSW, K33 KEYSW, K34 KEYSW, K35 KEYSW, K36 KEYSW, K37 KEYSW, K38 KEYSW, K39 KEYSW, K4 KEYSW, K40 KEYSW, K41 KEYSW, K42 KEYSW, K43 KEYSW, K44 KEYSW, K45 KEYSW, K46 KEYSW, K47 KEYSW, K48 KEYSW, K49 KEYSW, K5 KEYSW, K50 KEYSW, K51 KEYSW, K52 KEYSW, K53 KEYSW, K54 KEYSW, K55 KEYSW, K56 KEYSW, K57 KEYSW, K58 KEYSW, K59 KEYSW, K6 KEYSW, K60 KEYSW, K61 KEYSW, K62 KEYSW, K63 KEYSW, K64 KEYSW, K65 KEYSW, K66 KEYSW, K67 KEYSW, K68 KEYSW, K7 KEYSW, K8 KEYSW, K9 KEYSW, SW1 Reset SW, U1 ATmega32A-A, Y1 16MHz

Commit message: Added fuses, column and diode wirings
Parts:
- added F1: 500mA, Fuse:Fuse_0805_2012Metric_Pad1.15x1.40mm_HandSolder, F.Cu at (96.0, 103.1)
- R2: moved to B.Cu
- moved R2 14.5 mm to (81.8, 123.2), turned to 0 degrees
- moved C6 7.73 mm to (159.5, 193.0)
- moved C7 3.57 mm to (179.3, 196.6)
- moved R3 3.54 mm to (100.3, 126.0), turned to 0 degrees
- moved U1 1.80 mm to (171.2, 189.7), turned to 45 degrees
- moved D1 1.78 mm to (94.7, 123.2)
- moved R4 0.76 mm to (100.3, 128.0), turned to 180 degrees
- moved D2 0.51 mm to (98.3, 123.2)
Connections:
- J2 pad A4: +5V -> Net-(J2-PadA4)
- J2 pad A9: +5V -> Net-(J2-PadA4)
- J2 pad B4: +5V -> Net-(J2-PadA4)
- J2 pad B9: +5V -> Net-(J2-PadA4)
- U1 pad 13: unconnected-(U1-Pad13) -> /Switch Matrix/COL0
- U1 pad 14: unconnected-(U1-Pad14) -> /Switch Matrix/COL1
- U1 pad 16: unconnected-(U1-Pad16) -> /Switch Matrix/COL2
- U1 pad 19: /Switch Matrix/COL8 -> /Switch Matrix/COL3
- U1 pad 20: /Switch Matrix/COL9 -> /Switch Matrix/COL4
- U1 pad 21: /Switch Matrix/COL10 -> /Switch Matrix/ROW1
- U1 pad 22: /Switch Matrix/COL11 -> /Switch Matrix/ROW2
- U1 pad 23: /Switch Matrix/COL12 -> /Switch Matrix/ROW3
- U1 pad 24: /Switch Matrix/COL13 -> /Switch Matrix/ROW4
- U1 pad 25: /Switch Matrix/COL14 -> /Switch Matrix/COL5
- U1 pad 26: /Switch Matrix/COL15 -> /Switch Matrix/COL6
- U1 pad 30: /Switch Matrix/COL2 -> /Switch Matrix/COL7
- U1 pad 31: /Switch Matrix/COL1 -> /Switch Matrix/COL8
- U1 pad 32: /Switch Matrix/COL0 -> /Switch Matrix/COL9
- U1 pad 33: /Switch Matrix/ROW4 -> /Switch Matrix/COL14
- U1 pad 34: /Switch Matrix/ROW3 -> /Switch Matrix/COL13
- U1 pad 35: /Switch Matrix/ROW2 -> /Switch Matrix/COL12
- U1 pad 36: /Switch Matrix/ROW1 -> /Switch Matrix/COL11
- U1 pad 37: /Switch Matrix/ROW0 -> /Switch Matrix/COL10
- U1 pad 40: /Switch Matrix/COL3 -> /Switch Matrix/COL15
- U1 pad 41: /Switch Matrix/COL4 -> unconnected-(U1-Pad41)
- U1 pad 42: /Switch Matrix/COL5 -> unconnected-(U1-Pad42)
- U1 pad 43: /Switch Matrix/COL6 -> unconnected-(U1-Pad43)
- U1 pad 44: /Switch Matrix/COL7 -> unconnected-(U1-Pad44)
- U1 pad 9: unconnected-(U1-Pad9) -> /Switch Matrix/ROW0
Routing:
- net /Switch Matrix/ROW0: track 0.00 -> 339.2 mm, vias 0 -> 2
- net /Switch Matrix/COL3: track 0.00 -> 91.0 mm
- net /Switch Matrix/COL11: track 0.00 -> 88.0 mm
- net /Switch Matrix/COL10: track 0.00 -> 88.0 mm
- net /Switch Matrix/COL6: track 0.00 -> 87.0 mm
- net /Switch Matrix/COL12: track 0.00 -> 84.1 mm
- net /Switch Matrix/COL13: track 0.00 -> 82.7 mm
- net /Switch Matrix/COL14: track 0.00 -> 80.4 mm
- net /Switch Matrix/COL15: track 0.00 -> 76.2 mm
- net /Switch Matrix/COL8: track 0.00 -> 67.0 mm
- net /Switch Matrix/COL5: track 0.00 -> 67.0 mm
- net /Switch Matrix/COL9: track 0.00 -> 67.0 mm
- net /Switch Matrix/COL4: track 0.00 -> 67.0 mm
- net /Switch Matrix/COL7: track 0.00 -> 67.0 mm
- net Net-(C2-Pad1): track 20.1 -> 2.81 mm
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- removed copper zone on F.Cu, net +5V
- removed copper zone on B.Cu, net GND
Other:
- board size 301 x 94.7 mm -> 301 x 97.3 mm

Commit message: Completed first pass at v1 board
Parts:
- C7: moved to B.Cu
- moved C5 123.4 mm to (189.2, 188.0)
- moved Y1 39.4 mm to (146.3, 193.8), turned to 90 degrees
- moved C2 39.2 mm to (151.1, 197.6)
- moved C1 38.7 mm to (151.1, 189.7)
- moved C6 5.41 mm to (163.7, 196.5), turned to 180 degrees
- moved SW1 3.89 mm to (236.7, 186.4), turned to 90 degrees
- moved C7 2.82 mm to (181.5, 194.8), turned to 0 degrees
- moved F1 1.85 mm to (95.5, 104.9), turned to 180 degrees
- moved J1 1.85 mm to (221.2, 184.4)
- moved C4 1.73 mm to (163.2, 182.9), turned to 135 degrees
- moved C3 0.93 mm to (178.5, 182.5), turned to 45 degrees
- moved R1 0.80 mm to (228.6, 185.4), turned to -90 degrees
- moved R5 0.25 mm to (91.2, 117.6)
Connections:
- U1 pad 21: /Switch Matrix/ROW1 -> /Switch Matrix/ROW3
- U1 pad 23: /Switch Matrix/ROW3 -> /Switch Matrix/ROW1
- U1 pad 24: /Switch Matrix/ROW4 -> /Switch Matrix/ROW0
- U1 pad 33: /Switch Matrix/COL14 -> /Switch Matrix/COL10
- U1 pad 34: /Switch Matrix/COL13 -> /Switch Matrix/COL11
- U1 pad 36: /Switch Matrix/COL11 -> /Switch Matrix/COL13
- U1 pad 37: /Switch Matrix/COL10 -> /Switch Matrix/COL14
- U1 pad 9: /Switch Matrix/ROW0 -> /Switch Matrix/ROW4
Routing:
- net /Switch Matrix/ROW1: track 0.00 -> 399.1 mm, vias 0 -> 4
- net /Switch Matrix/ROW2: track 0.00 -> 360.6 mm, vias 0 -> 4
- net /Switch Matrix/ROW3: track 0.00 -> 329.5 mm, vias 0 -> 4
- net /Switch Matrix/ROW4: track 0.00 -> 322.6 mm
- net /Switch Matrix/COL15: track 76.2 -> 292.7 mm
- net /Switch Matrix/COL14: track 80.4 -> 268.1 mm, vias 0 -> 1
- net /Switch Matrix/COL13: track 82.7 -> 250.3 mm, vias 0 -> 1
- net /Switch Matrix/COL12: track 84.1 -> 231.9 mm, vias 0 -> 1
- net /Switch Matrix/COL11: track 88.0 -> 216.1 mm, vias 0 -> 1
- net /Switch Matrix/COL10: track 88.0 -> 198.1 mm, vias 0 -> 1
- net /Switch Matrix/COL9: track 67.0 -> 172.7 mm, vias 0 -> 1
- net /Switch Matrix/COL8: track 67.0 -> 153.5 mm, vias 0 -> 1
- net /Switch Matrix/COL0: track 85.1 -> 167.8 mm, vias 0 -> 1
- net /RST: track 0.00 -> 81.7 mm, vias 0 -> 1
- net /Switch Matrix/ROW0: track 339.2 -> 408.2 mm, vias 2 -> 4
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- added copper zone on F.Cu, net +5V
- added copper zone on B.Cu, net GND
Other:
- outline, holes or cut-outs redrawn

Commit message: Final V1 Board, Ordered
Parts:
- added ?: LOGO, keyboard_parts:guy, B.Cu at (361.6, 118.0)
- added ?: LOGO, keyboard_parts:dollEr, B.Cu at (96.2, 186.1)
- moved C6 1.68 mm to (165.4, 196.6)
- moved C4 1.40 mm to (164.6, 182.9)
- moved Y1 1.27 mm to (145.0, 193.8)
- moved C1 1.02 mm to (150.1, 189.7)
- moved C2 1.02 mm to (150.1, 197.6)
Routing:
- net /Switch Matrix/COL1: track 134.1 -> 145.0 mm
- net /D-: track 120.4 -> 112.0 mm
- net /D+: track 120.3 -> 111.9 mm
- net /Switch Matrix/ROW3: track 329.5 -> 334.8 mm
- net +5V: track 44.6 -> 42.3 mm
- net Net-(C2-Pad1): track 25.9 -> 27.4 mm
- net Net-(C1-Pad1): track 25.1 -> 26.6 mm
- net GND: track 37.6 -> 38.0 mm, vias 3 -> 5
Other:
- board text added: "1"
- board text added: "D:"
